File: electrical-schematic/1DOF_FOC_Force-Feedback.kicad_sch (KiCad schematic)
At the start: 8 parts, among them U4 AS5047P ADAPTERBOARD, U5 AS5047P ADAPTERBOARD, U6 GBM2804, U8 GBM2804

Commit message: Updated to use quadrature for encoders
Connections:
- net GND: no longer U5.6 (TEST)
- net at U5.10 (A): now also U7.8 (A)
- net at U5.11 (I_PWM): now also U7.10 (I/PWM)
- net at U5.3 (CSn): no longer U7.11 (SPI_CS)
- net at U1.1 (CAN_H), U2.3 (CAN_H), U7.3 (CAN_H): no longer U5.4 (CLK), U7.10 (SPI_CLK)
- net at U1.2 (CAN_L), U2.4 (CAN_L), U7.4 (CAN_L): no longer U5.5 (MOSI), U7.8 (SPI_MOSI)
- net at U5.7 (MISO): no longer U7.9 (SPI_MISO)
- net at U5.9 (B): now also U7.9 (B)
- net at U4.10 (A): now also U2.8 (A)
- net at U4.11 (I_PWM): now also U2.10 (I/PWM)
- net at U4.3 (CSn): no longer U2.11 (SPI_CS)
- net at U4.4 (CLK): no longer U2.10 (SPI_CLK)
- net at U4.5 (MOSI): no longer U2.8 (SPI_MOSI)
- net at U4.7 (MISO): no longer U2.9 (SPI_MISO)
- net at U4.9 (B): now also U2.9 (B)
